Commit message: Rename `_publishers` to `gripper_pubs` for clarity and update SRDF with updated gripper group joints and full collision matrix for Robotiq 2F-85
--Moveit Package regenerated

File: dual_arm_moveit_config/config/dual_ur5e.ros2_control.xacro (robot description, xacro)
@@ -92,4 +92,18 @@
                 <state_interface name="velocity"/>
             </joint>
+            <joint name="left_robotiq_85_left_knuckle_joint">
+                <command_interface name="position"/>
+                <state_interface name="position">
+                  <param name="initial_value">${initial_positions['left_robotiq_85_left_knuckle_joint']}</param>
+                </state_interface>
+                <state_interface name="velocity"/>
+            </joint>
+            <joint name="right_robotiq_85_left_knuckle_joint">
+                <command_interface name="position"/>
+                <state_interface name="position">
+                  <param name="initial_value">${initial_positions['right_robotiq_85_left_knuckle_joint']}</param>
+                </state_interface>
+                <state_interface name="velocity"/>
+            </joint>
         </ros2_control>
     </xacro:macro>
