Commit message: Add gripper bridge node and integrate Robotiq 2F-85 grippers into dual-arm setup
- Implement `gripper_bridge_node` to convert normalized 0–1 targets to `JointTrajectory` commands for Robotiq grippers
- Extend SRDF with gripper planning groups, end-effectors, and comprehensive collision exclusions (including adapter and gripper internals)
- Configure gripper `joint_trajectory_controller` instances in `ros2_controllers.yaml` and `moveit_controllers.yaml`
- Update URDF.xacro to include Robotiq adapter and gripper macros for both arms
- Add gripper controller entries to `setup.py` entry points

-- Not working yet

File: dual_arm_description/urdf/dual_arm.urdf.xacro (robot description, xacro)
@@ -1,9 +1,13 @@
 <?xml version="1.0"?>
 <robot xmlns:xacro="http://wiki.ros.org/xacro" name="dual_ur5e">
-  <!-- Import UR5e Macro -->
+  <!-- ── Arm macro ─────────────────────────────────────────────────────── -->
   <xacro:include filename="$(find ur_description)/urdf/ur_macro.xacro"/>
-  <!-- World Link -->
+  <!-- ── Gripper macros ────────────────────────────────────────────────── -->
+  <!-- robotiq_gripper: attaches gripper geometry + its own ros2_control block -->
+  <xacro:include filename="$(find robotiq_description)/urdf/robotiq_2f_85_macro.urdf.xacro"/>
+  <!-- ur_to_robotiq: inserts the physical UR-to-Robotiq adapter link + mesh  -->
+  <xacro:include filename="$(find robotiq_description)/urdf/ur_to_robotiq_adapter.urdf.xacro"/>
+  <!-- ── World & table ─────────────────────────────────────────────────── -->
   <link name="world"/>
-  <!-- Simple Table/Base -->
   <link name="base_table">
     <visual>
@@ -11,4 +15,7 @@
       <material name="gray"><color rgba="0.5 0.5 0.5 1.0"/></material>
     </visual>
+    <collision>
+      <geometry><box size="1.0 2.0 0.1"/></geometry>
+    </collision>
   </link>
   <joint name="world_to_table" type="fixed">
@@ -17,4 +24,5 @@
     <origin xyz="0 0 0.8" rpy="0 0 0"/>
   </joint>
+  <!-- ── Left arm ──────────────────────────────────────────────────────── -->
   <xacro:ur_robot
     name="left_arm"
@@ -22,5 +30,11 @@
     parent="base_table"
     use_fake_hardware="true"
-    initial_positions="${dict(shoulder_pan_joint=0.0,shoulder_lift_joint=-1.57,elbow_joint=0.0,wrist_1_joint=-1.57,wrist_2_joint=0.0,wrist_3_joint=0.0)}"
+    initial_positions="${dict(
+      shoulder_pan_joint=0.4,
+      shoulder_lift_joint=-1.2,
+      elbow_joint=1.8,
+      wrist_1_joint=-2.2,
+      wrist_2_joint=-1.57,
+      wrist_3_joint=0.0)}"
     joint_limits_parameters_file="$(find ur_description)/config/ur5e/joint_limits.yaml"
     kinematics_parameters_file="$(find ur_description)/config/ur5e/default_kinematics.yaml"
@@ -29,4 +43,22 @@
     <origin xyz="0 0.4 0.05" rpy="0 0 0" />
   </xacro:ur_robot>
+  <!-- Left adapter: inserts the UR-to-Robotiq coupler mesh between
+       left_tool0 and a new mount link (left_gripper_mount).
+       The adapter macro creates left_gripper_mount as an empty link. -->
+  <xacro:ur_to_robotiq
+    prefix="left_"
+    parent="left_tool0"
+    child="left_gripper_mount"/>
+  <!-- Left gripper: attached to left_gripper_mount.
+       use_fake_hardware=true makes the macro add its own mock ros2_control
+       system for left_finger_joint — no manual joint entry needed. -->
+  <xacro:robotiq_gripper
+    name="left_RobotiqGripper"
+    prefix="left_"
+    parent="left_gripper_mount"
+    use_fake_hardware="true">
+    <origin xyz="0 0 0" rpy="0 0 0"/>
+  </xacro:robotiq_gripper>
+  <!-- ── Right arm ─────────────────────────────────────────────────────── -->
   <xacro:ur_robot
     name="right_arm"
@@ -34,5 +66,11 @@
     parent="base_table"
     use_fake_hardware="true"
-    initial_positions="${dict(shoulder_pan_joint=0.0,shoulder_lift_joint=-1.57,elbow_joint=0.0,wrist_1_joint=-1.57,wrist_2_joint=0.0,wrist_3_joint=0.0)}"
+    initial_positions="${dict(
+      shoulder_pan_joint=-0.4,
+      shoulder_lift_joint=-1.2,
+      elbow_joint=1.8,
+      wrist_1_joint=-2.2,
+      wrist_2_joint=1.57,
+      wrist_3_joint=0.0)}"
     joint_limits_parameters_file="$(find ur_description)/config/ur5e/joint_limits.yaml"
     kinematics_parameters_file="$(find ur_description)/config/ur5e/default_kinematics.yaml"
@@ -41,3 +79,16 @@
     <origin xyz="0 -0.4 0.05" rpy="0 0 0" />
   </xacro:ur_robot>
+  <!-- Right adapter -->
+  <xacro:ur_to_robotiq
+    prefix="right_"
+    parent="right_tool0"
+    child="right_gripper_mount"/>
+  <!-- Right gripper -->
+  <xacro:robotiq_gripper
+    name="right_RobotiqGripper"
+    prefix="right_"
+    parent="right_gripper_mount"
+    use_fake_hardware="true">
+    <origin xyz="0 0 0" rpy="0 0 0"/>
+  </xacro:robotiq_gripper>
 </robot>

Commit message: Add handover baton visualization marker and safety latch for teleop robustness
- Introduce `handover_baton_node` to publish a neon-green cylinder marker at configurable pose for handover demo
- Update RViz config to display baton marker and extend launch files with parameters and conditional node
- Implement safety latch in `teleop_node`: pause commands and lock control on hard Servo stops (status 2, 4, 5)
- Add parameters: `safety_latch_enabled`, `split_control_window`, `invert_lateral_axis`, `swap_control_panes`
- Refactor control coordinate mapping to support pane-based input zones with intuitive lateral mapping
- Improve debug overlay with per-arm panes and annotations
- Fix right arm wrist2 default joint angle in URDF and initial positions

File: dual_arm_description/urdf/dual_arm.urdf.xacro (robot description, xacro)
@@ -12,9 +12,9 @@
   <link name="base_table">
     <visual>
-      <geometry><box size="1.0 2.0 0.1"/></geometry>
+      <geometry><box size="2.0 2.0 0.1"/></geometry>
       <material name="gray"><color rgba="0.5 0.5 0.5 1.0"/></material>
     </visual>
     <collision>
-      <geometry><box size="1.0 2.0 0.1"/></geometry>
+      <geometry><box size="2.0 2.0 0.1"/></geometry>
     </collision>
   </link>
@@ -22,5 +22,5 @@
     <parent link="world"/>
     <child link="base_table"/>
-    <origin xyz="0 0 0.8" rpy="0 0 0"/>
+    <origin xyz="0 0 0.5" rpy="0 0 0"/>
   </joint>
   <!-- ── Left arm ──────────────────────────────────────────────────────── -->
@@ -72,5 +72,5 @@
       elbow_joint=1.8,
       wrist_1_joint=-2.2,
-      wrist_2_joint=1.57,
+      wrist_2_joint=-1.57,
       wrist_3_joint=0.0)}"
     joint_limits_parameters_file="$(find ur_description)/config/ur5e/joint_limits.yaml"
